Commit message: move arm to table and cube scaled 50%

File: src/robots/asimov/urdf/ASIMOV_FINAL_2.urdf (robot description, URDF)
Before this commit: robot asimov, 5 links, 4 joints
Links:
- link FL_wheel: geometry collision cylinder length=0.048 radius=0.075; visual mesh filename=package://asimov/meshes/decimated/FL_wheel.STL
- link FR_wheel: geometry collision cylinder length=0.048 radius=0.075; visual mesh filename=package://asimov/meshes/decimated/FR_wheel.STL
- link RL_wheel: geometry collision cylinder length=0.048 radius=0.075; visual mesh filename=package://asimov/meshes/decimated/RL_wheel.STL
- link RR_wheel: geometry collision cylinder length=0.048 radius=0.075; visual mesh filename=package://asimov/meshes/decimated/RR_wheel.STL
- link base_link: geometry collision box size=0.75 0.55 0.26; visual mesh filename=package://asimov/meshes/decimated/base_link.STL
