Commit message: add cameera t oend effector

File: src/robots/mini_arm_ros2/urdf/mini_arm.urdf (robot description, URDF)
Before this commit: robot mini_arm_ros2, 14 links, 13 joints
Links:
- added link camera_link, mass 0.01; collision box size=0.02 0.02 0.02; visual box size=0.02 0.02 0.02
Joints:
- added joint camera_joint: type fixed, parent end_base, child camera_link, origin xyz=0.05 0 0.02 rpy=0 0.3 0

Commit message: Scaled up arm and created urdf for model

File: src/robots/mini_arm_ros2/urdf/mini_arm.urdf (robot description, URDF)
Before this commit: robot mini_arm_ros2, 15 links, 14 joints
Links:
- removed link anchor_left
- removed link anchor_right
- link base_link: mass 0.0763754463040628 -> 1.1921875000000002; geometry collision box size=0.4 0.2 0.22499999999999998; visual mesh filename=package://mini_arm_ros2/meshes/decimated/base_link.STL scale=2.5 2.5 2.5
- link base_rotator: mass 0.0393066448790151 -> 0.6140625000000001; geometry collision cylinder length=0.0625 radius=0.05; visual mesh filename=package://mini_arm_ros2/meshes/decimated/base_rotator.STL scale=2.5 2.5 2.5
- link camera_link: mass 0.01 -> 0.15625; geometry collision box size=0.05 0.05 0.05; visual box size=0.05 0.05 0.05
- link elbow_Link: mass 0.0420586657729736 -> 0.65625; geometry collision box size=0.25 0.075 0.025; visual mesh filename=package://mini_arm_ros2/meshes/decimated/elbow_Link.STL scale=2.5 2.5 2.5
- link end_base: mass 0.0345345547168646 -> 0.5390625; geometry collision box size=0.1375 0.1 0.05; visual mesh filename=package://mini_arm_ros2/meshes/decimated/end_base.STL scale=2.5 2.5 2.5
- link finger_left: mass 0.00220506613383814 -> 0.034375; geometry collision box size=0.1 0.025 0.0125; visual mesh filename=package://mini_arm_ros2/meshes/decimated/finger_left.STL scale=2.5 2.5 2.5
- link finger_right: mass 0.00221856156382406 -> 0.034375; geometry collision box size=0.1 0.025 0.0125; visual mesh filename=package://mini_arm_ros2/meshes/decimated/finger_right.STL scale=2.5 2.5 2.5
- link gear_left: mass 0.00146187481822585 -> 0.021875000000000002; geometry collision box size=0.075 0.025 0.0125; visual mesh filename=package://mini_arm_ros2/meshes/decimated/gear_left.STL scale=2.5 2.5 2.5
- link gear_right: mass 0.00207956891883696 -> 0.03125; geometry collision box size=0.075 0.025 0.0125; visual mesh filename=package://mini_arm_ros2/meshes/decimated/gear_right.STL scale=2.5 2.5 2.5
- link shoulder_link: mass 0.0144514859726596 -> 0.22499999999999998; geometry collision box size=0.05 0.05 0.25; visual mesh filename=package://mini_arm_ros2/meshes/decimated/shoulder_link.STL scale=2.5 2.5 2.5
- link wrist_Link: mass 0.0644141323115809 -> 1.00625; geometry collision box size=0.1375 0.1 0.075; visual mesh filename=package://mini_arm_ros2/meshes/decimated/wrist_Link.STL scale=2.5 2.5 2.5
Joints:
- removed joint anchor_left_joint
- removed joint anchor_right_joint
- removed joint world_fixed
- added joint base_joint: type fixed, parent world, child base_link, origin xyz=0 0 0 rpy=0 0 0
- joint base_rotator_joint: origin xyz=-0.15562 -0.016822 -0.042262 rpy=0 0 -0.28913 -> xyz=-0.38905 -0.042055 -0.105655 rpy=0 0 -0.28913
- joint camera_joint: origin xyz=0.05 0 0.02 rpy=0 0.3 0 -> xyz=0.125 0 0.05 rpy=0 0.3 0
- joint elbow_joint: axis -0.134583598084368 0.990902242971861 0 -> -0.13458 0.9909 0; origin xyz=-0.000720890128520002 0.0027573206963649 0.103 rpy=0.109466615902697 -0.677396307197321 0.0821328070422031 -> xyz=-0.0018000000000000002 0.006874999999999999 0.2575 rpy=0.10946 -0.67739 0.08213
- joint end_joint: origin xyz=0.0545990000041253 0.0259989999957502 0.0269999999957503 rpy=0.0529233606550124 0 0 -> xyz=0.1364975 0.0649975 0.0674975 rpy=0.05292 0 0
- joint finger_left_joint: origin xyz=0.030762 0 0 rpy=0 0 -0.68869 -> xyz=0.076905 0 0 rpy=0 0 -0.68869
- joint finger_right_joint: origin xyz=0.030762 0 0.0025 rpy=0 0 0.98133 -> xyz=0.076905 0 0.00625 rpy=0 0 0.98133
- joint gear_left_joint: origin xyz=0.0305 0.01226 0.0068 rpy=0 0 0.3732 -> xyz=0.07625 0.03065 0.016999999999999998 rpy=0 0 0.3732
- joint gear_right_joint: origin xyz=0.03 -0.015741 0.0043 rpy=0 0 -0.60373 -> xyz=0.075 -0.03924999999999999 0.01075 rpy=0 0 -0.60373
- joint shoulder_joint: origin xyz=0.001501 -0.0236 0.0201 rpy=0.12148 -0.43402 -0.28254 -> xyz=0.0037524999999999998 -0.059 0.05025 rpy=0.12148 -0.43402 -0.28254
- joint tool0_fixed: origin xyz=0.10 0 0 rpy=0 0 0 -> xyz=0.25 0 0 rpy=0 0 0
- joint wrist_joint: origin xyz=0.0957085548832958 0.0123430961736119 0.00149999999999995 rpy=0 1.15689373274673 0.134993225634174 -> xyz=0.23925 0.03075 0.00375 rpy=0 1.15689 0.13499
