Commit message: scale dynamic to be proprtional to arm

File: src/robots/mini_arm_ros2/urdf/mini_arm.xacro (robot description, xacro)
@@ -57,5 +57,6 @@
       <child link="${prefix}base_rotator" />
       <axis xyz="0 0 -1" />
-      <limit lower="-1.57" upper="1.57" effort="1.0" velocity="2.0" />
+      <limit lower="-1.57" upper="1.57" effort="${20.0 * scale**4}" velocity="2.0" />
+      <dynamics damping="${0.5 * scale**4}" friction="${0.3 * scale**4}" />
     </joint>
     <link name="${prefix}shoulder_link">
@@ -85,5 +86,6 @@
       <child link="${prefix}shoulder_link" />
       <axis xyz="-0.25294 0.96748 0" />
-      <limit lower="-1.57" upper="1.57" effort="1.0" velocity="2.0" />
+      <limit lower="-1.57" upper="1.57" effort="${30.0 * scale**4}" velocity="2.0" />
+      <dynamics damping="${1.0 * scale**4}" friction="${0.5 * scale**4}" />
     </joint>
     <link name="${prefix}elbow_Link">
@@ -113,5 +115,6 @@
       <child link="${prefix}elbow_Link" />
       <axis xyz="-0.13458 0.9909 0" />
-      <limit lower="-1.57" upper="1.57" effort="1.0" velocity="2.0" />
+      <limit lower="-1.57" upper="1.57" effort="${25.0 * scale**4}" velocity="2.0" />
+      <dynamics damping="${0.8 * scale**4}" friction="${0.4 * scale**4}" />
     </joint>
     <link name="${prefix}wrist_Link">
@@ -141,5 +144,6 @@
       <child link="${prefix}wrist_Link" />
       <axis xyz="0 1 0" />
-      <limit lower="-1.57" upper="1.57" effort="1.0" velocity="2.0" />
+      <limit lower="-1.57" upper="1.57" effort="${15.0 * scale**4}" velocity="2.0" />
+      <dynamics damping="${0.5 * scale**4}" friction="${0.3 * scale**4}" />
     </joint>
     <link name="${prefix}end_base">
@@ -169,5 +173,6 @@
       <child link="${prefix}end_base" />
       <axis xyz="-1 0 0" />
-      <limit lower="-1.57" upper="1.57" effort="1.0" velocity="2.0" />
+      <limit lower="-1.57" upper="1.57" effort="${10.0 * scale**4}" velocity="2.0" />
+      <dynamics damping="${0.4 * scale**4}" friction="${0.2 * scale**4}" />
     </joint>
     <!-- Simplified Gripper -->
@@ -196,5 +201,6 @@
       <child link="${prefix}gear_right" />
       <axis xyz="0 0 -1" />
-      <limit lower="-1.57" upper="1.57" effort="1.0" velocity="2.0" />
+      <limit lower="-1.57" upper="1.57" effort="${5.0 * scale**4}" velocity="2.0" />
+      <dynamics damping="${0.3 * scale**4}" friction="${0.2 * scale**4}" />
     </joint>
     <link name="${prefix}finger_right">
@@ -222,5 +228,6 @@
       <child link="${prefix}finger_right" />
       <axis xyz="0 0 1" />
-      <limit lower="-1.57" upper="1.57" effort="1.0" velocity="2.0" />
+      <limit lower="-1.57" upper="1.57" effort="${5.0 * scale**4}" velocity="2.0" />
+      <dynamics damping="${0.3 * scale**4}" friction="${0.2 * scale**4}" />
       <mimic joint="${prefix}gear_right_joint" multiplier="1" offset="0" />
     </joint>
@@ -249,5 +256,6 @@
       <child link="${prefix}gear_left" />
       <axis xyz="0 0 -1" />
-      <limit lower="-1.57" upper="1.57" effort="1.0" velocity="2.0" />
+      <limit lower="-1.57" upper="1.57" effort="${5.0 * scale**4}" velocity="2.0" />
+      <dynamics damping="${0.3 * scale**4}" friction="${0.2 * scale**4}" />
       <mimic joint="${prefix}gear_right_joint" multiplier="-1" offset="0" />
     </joint>
@@ -276,5 +284,6 @@
       <child link="${prefix}finger_left" />
       <axis xyz="0 0 1" />
-      <limit lower="-1.57" upper="1.57" effort="1.0" velocity="2.0" />
+      <limit lower="-1.57" upper="1.57" effort="${5.0 * scale**4}" velocity="2.0" />
+      <dynamics damping="${0.3 * scale**4}" friction="${0.2 * scale**4}" />
       <mimic joint="${prefix}gear_right_joint" multiplier="-1" offset="0" />
     </joint>
@@ -327,4 +336,5 @@
           </clip>
         </camera>
+        <topic>arm_camera/image_raw</topic>
       </sensor>
     </gazebo>
