Commit message: bridge ros2 and gazebo

File: src/robots/full_arm_ros2/urdf/diffbot_ros2_control.xacro (robot description, xacro)
@@ -4,5 +4,10 @@
     <ros2_control name="${name}" type="system">
       <hardware>
-        <plugin>mock_components/GenericSystem</plugin>
+        <xacro:if value="${sim == 'gz'}">
+          <plugin>ign_ros2_control/IgnitionSystem</plugin>
+        </xacro:if>
+        <xacro:if value="${sim != 'gz'}">
+          <plugin>mock_components/GenericSystem</plugin>
+        </xacro:if>
       </hardware>
       <joint name="${prefix}fl_wheel_joint">

File: src/robots/full_arm_ros2/urdf/full_arm_ros2.urdf.xacro (robot description, xacro)
@@ -1,4 +1,5 @@
 <?xml version="1.0"?>
 <robot name="full_arm_ros2" xmlns:xacro="http://www.ros.org/wiki/xacro">
+  <xacro:arg name="sim" default="true"/>
   <!-- Include the arm macro -->
   <xacro:include filename="$(find mini_arm_ros2)/urdf/mini_arm.xacro" />
@@ -77,6 +78,78 @@
     <origin xyz="0.18 -0.21 0.34" rpy="0 0 0" />
   </xacro:mini_arm>
-  <!-- Combine ROS2 Control -->
-  <xacro:diffbot_ros2_control name="base_control" prefix="" sim="true"/>
-  <xacro:mini_arm_ros2_control name="arm_control" prefix="arm_"/>
+  <!-- Single combined ROS2 Control (ign_ros2_control on Humble needs one hardware system) -->
+  <ros2_control name="full_robot_control" type="system">
+    <hardware>
+      <xacro:if value="${'$(arg sim)' == 'gz'}">
+        <plugin>ign_ros2_control/IgnitionSystem</plugin>
+      </xacro:if>
+      <xacro:if value="${'$(arg sim)' != 'gz'}">
+        <plugin>mock_components/GenericSystem</plugin>
+      </xacro:if>
+    </hardware>
+    <!-- Wheels (velocity control) -->
+    <joint name="fl_wheel_joint">
+      <command_interface name="velocity"/>
+      <state_interface name="position"/>
+      <state_interface name="velocity"/>
+    </joint>
+    <joint name="fr_wheel_joint">
+      <command_interface name="velocity"/>
+      <state_interface name="position"/>
+      <state_interface name="velocity"/>
+    </joint>
+    <joint name="rl_wheel_joint">
+      <command_interface name="velocity"/>
+      <state_interface name="position"/>
+      <state_interface name="velocity"/>
+    </joint>
+    <joint name="rr_wheel_joint">
+      <command_interface name="velocity"/>
+      <state_interface name="position"/>
+      <state_interface name="velocity"/>
+    </joint>
+    <!-- Arm (position control) -->
+    <joint name="arm_base_rotator_joint">
+      <command_interface name="position"/>
+      <state_interface name="position"/>
+    </joint>
+    <joint name="arm_shoulder_joint">
+      <command_interface name="position"/>
+      <state_interface name="position"/>
+    </joint>
+    <joint name="arm_elbow_joint">
+      <command_interface name="position"/>
+      <state_interface name="position"/>
+    </joint>
+    <joint name="arm_wrist_joint">
+      <command_interface name="position"/>
+      <state_interface name="position"/>
+    </joint>
+    <joint name="arm_end_joint">
+      <command_interface name="position"/>
+      <state_interface name="position"/>
+    </joint>
+    <joint name="arm_gear_right_joint">
+      <command_interface name="position"/>
+      <state_interface name="position"/>
+    </joint>
+    <!-- Gripper mimic joints (state only, URDF mimic tags handle physics) -->
+    <joint name="arm_gear_left_joint">
+      <state_interface name="position"/>
+    </joint>
+    <joint name="arm_finger_right_joint">
+      <state_interface name="position"/>
+    </joint>
+    <joint name="arm_finger_left_joint">
+      <state_interface name="position"/>
+    </joint>
+  </ros2_control>
+  <!-- Gazebo ros2_control plugin (only meaningful when sim:=gz) -->
+  <xacro:if value="${'$(arg sim)' == 'gz'}">
+    <gazebo>
+      <plugin filename="ign_ros2_control-system" name="ign_ros2_control::IgnitionROS2ControlPlugin">
+        <parameters>$(find full_arm_ros2)/config/combined_controllers.yaml</parameters>
+      </plugin>
+    </gazebo>
+  </xacro:if>
 </robot>

File: src/robots/mini_arm_ros2/urdf/mini_arm.xacro (robot description, xacro)
@@ -311,8 +311,13 @@
     </joint>
   </xacro:macro>
-  <xacro:macro name="mini_arm_ros2_control" params="name prefix">
+  <xacro:macro name="mini_arm_ros2_control" params="name prefix sim:=true">
     <ros2_control name="${name}" type="system">
       <hardware>
-        <plugin>mock_components/GenericSystem</plugin>
+        <xacro:if value="${sim == 'gz'}">
+          <plugin>ign_ros2_control/IgnitionSystem</plugin>
+        </xacro:if>
+        <xacro:if value="${sim != 'gz'}">
+          <plugin>mock_components/GenericSystem</plugin>
+        </xacro:if>
       </hardware>
       <joint name="${prefix}base_rotator_joint">
@@ -341,17 +346,11 @@
       </joint>
       <joint name="${prefix}gear_left_joint">
-        <param name="mimic">${prefix}gear_right_joint</param>
-        <param name="multiplier">-1</param>
-        <command_interface name="position"/>
+        <state_interface name="position"/>
       </joint>
       <joint name="${prefix}finger_right_joint">
-        <param name="mimic">${prefix}gear_right_joint</param>
-        <param name="multiplier">1</param>
-        <command_interface name="position"/>
+        <state_interface name="position"/>
       </joint>
       <joint name="${prefix}finger_left_joint">
-        <param name="mimic">${prefix}gear_right_joint</param>
-        <param name="multiplier">-1</param>
-        <command_interface name="position"/>
+        <state_interface name="position"/>
       </joint>
     </ros2_control>
