Commit message: change urdf to decimate, add camera to arm

File: src/robots/full_arm_ros2/urdf/full_arm_ros2.urdf.xacro (robot description, xacro)
@@ -23,5 +23,5 @@
       <origin xyz="0 0 0" rpy="0 0 0"/>
       <geometry>
-        <mesh filename="package://full_arm_ros2/meshes/base_link.STL"/>
+        <mesh filename="package://full_arm_ros2/meshes/decimated/base_link.STL"/>
       </geometry>
       <material name="blue"/>
@@ -30,5 +30,5 @@
       <origin xyz="0 0 0" rpy="0 0 0"/>
       <geometry>
-        <mesh filename="package://full_arm_ros2/meshes/base_link.STL"/>
+        <mesh filename="package://full_arm_ros2/meshes/decimated/base_link.STL"/>
       </geometry>
     </collision>
@@ -45,5 +45,5 @@
         <origin xyz="0 0 0" rpy="0 0 0"/>
         <geometry>
-          <mesh filename="package://full_arm_ros2/meshes/${prefix}_wheel.STL"/>
+          <mesh filename="package://full_arm_ros2/meshes/decimated/${prefix}_wheel.STL"/>
         </geometry>
         <material name="wheel_gray"/>
@@ -52,5 +52,5 @@
         <origin xyz="0 0 0" rpy="0 0 0"/>
         <geometry>
-          <mesh filename="package://full_arm_ros2/meshes/${prefix}_wheel.STL"/>
+          <mesh filename="package://full_arm_ros2/meshes/decimated/${prefix}_wheel.STL"/>
         </geometry>
       </collision>

File: src/robots/mini_arm_ros2/urdf/mini_arm.xacro (robot description, xacro)
@@ -310,4 +310,23 @@
       <origin xyz="${0.05 * scale} 0 ${0.02 * scale}" rpy="0 0.3 0"/>
     </joint>
+    <!-- Gazebo camera sensor -->
+    <gazebo reference="${prefix}camera_link">
+      <sensor name="arm_camera" type="camera">
+        <always_on>true</always_on>
+        <update_rate>15</update_rate>
+        <camera>
+          <horizontal_fov>1.047</horizontal_fov>
+          <image>
+            <width>640</width>
+            <height>480</height>
+            <format>R8G8B8</format>
+          </image>
+          <clip>
+            <near>0.01</near>
+            <far>10.0</far>
+          </clip>
+        </camera>
+      </sensor>
+    </gazebo>
   </xacro:macro>
   <xacro:macro name="mini_arm_ros2_control" params="name prefix sim:=true">
